File: hardware/rev_a/BalanceBoard/BalanceBoard.kicad_pcb (KiCad board)
At the start: 2 copper layers, 45 x 22 mm, 54 parts, among them J1 48037-0001, J2 5103309-1, J3 2212S-04SG-85, T00 TestPoints, T01 TestPoints, T02 TestPoints, T03 TestPoints, T04 TestPoints, T05 TestPoints, T06 TestPoints, T07 TestPoints, T10 TestPoints, T11 TestPoints, T12 TestPoints, T13 TestPoints, T14 TestPoints, T15 TestPoints, T16 TestPoints, T17 TestPoints, T21 TestPoints, T31 TestPoints, T32 TestPoints, T33 TestPoints, T40 TestPoints, T41 TestPoints, T42 TestPoints, T43 TestPoints, T44 TestPoints, T45 TestPoints, T46 TestPoints, T47 TestPoints, T48 TestPoints, T49 TestPoints, T50 TestPoints, U1 C8051F850-A-GU, U2 FT232RL

Commit message: tidy
Connections:
- J2 pad 1: Net-(J2-Pad1) -> unconnected-(J2-Pad1)
- J2 pad 8: Net-(J2-Pad8) -> unconnected-(J2-Pad8)
- U1 pad 1: Net-(U1-Pad1) -> unconnected-(U1-Pad1)
- U1 pad 13: Net-(U1-Pad13) -> unconnected-(U1-Pad13)
- U1 pad 24: Net-(U1-Pad24) -> unconnected-(U1-Pad24)
- U2 pad 12: Net-(U2-Pad12) -> unconnected-(U2-Pad12)
- U2 pad 13: Net-(U2-Pad13) -> unconnected-(U2-Pad13)
- U2 pad 19: Net-(U2-Pad19) -> unconnected-(U2-Pad19)
- U2 pad 22: Net-(U2-Pad22) -> unconnected-(U2-Pad22)
- U2 pad 23: Net-(U2-Pad23) -> unconnected-(U2-Pad23)
- U2 pad 24: Net-(U2-Pad24) -> unconnected-(U2-Pad24)
- U2 pad 27: Net-(U2-Pad27) -> unconnected-(U2-Pad27)
- U2 pad 28: Net-(U2-Pad28) -> unconnected-(U2-Pad28)
- U2 pad 8: Net-(U2-Pad8) -> unconnected-(U2-Pad8)

Commit message: reset pcb
Parts:
- moved U2 38.1 mm to (76.0, 166.0)
- moved J3 18.2 mm to (68.1, 152.4)
- moved J2 16.7 mm to (70.4, 195.0)
- moved U1 12.8 mm to (51.1, 162.3)
- moved J1 10.8 mm to (27.2, 171.4)
Routing:
- net GND: track 112.0 -> 0.00 mm, vias 86 -> 0
- net +5V: track 72.6 -> 0.00 mm, vias 8 -> 0
- net +3V3: track 68.7 -> 0.00 mm, vias 1 -> 0
- net /RX: track 34.1 -> 0.00 mm, vias 1 -> 0
- net /FT_TO_MCU: track 29.9 -> 0.00 mm, vias 2 -> 0
- net /TCK_C2D: track 25.4 -> 0.00 mm, vias 1 -> 0
- net /TDI_C2CK: track 24.4 -> 0.00 mm, vias 1 -> 0
- net /MCU_TO_FT: track 24.2 -> 0.00 mm, vias 2 -> 0
- net Net-(R3-Pad1): track 16.9 -> 0.00 mm, vias 2 -> 0
- net Net-(T01-Pad1): track 16.4 -> 0.00 mm
- net Net-(T10-Pad1): track 15.2 -> 0.00 mm, vias 1 -> 0
- net Net-(T02-Pad1): track 13.7 -> 0.00 mm
- net /TDO_C2D: track 12.2 -> 0.00 mm
- net Net-(T17-Pad1): track 11.6 -> 0.00 mm
- net Net-(T00-Pad1): track 11.5 -> 0.00 mm
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- removed copper zone on F.Cu, net +3V3
- removed copper zone on B.Cu, net +5V
- removed copper zone on B.Cu, net GND
- removed copper zone on F.Cu, net GND
- removed copper zone on F.Cu, net VCC
Other:
- board outline removed

Commit message: change usb
Parts:
- removed C8: CAP_0603, receiver:0603
- removed J3: 2212S-04SG-85, receiver:2212S-04SG-85
- removed R8, R9: RES_0603, receiver:0603
- removed T50: TestPoints, receiver:TestPoint
- J1: value 48037-0001 -> 47491-0001-TR425; footprint receiver:48037-0001 -> receiver:47491-0001-TR425
- moved U1 23.9 mm to (69.5, 147.0), turned to 0 degrees
- moved J1 10.7 mm to (31.3, 161.5), turned to 0 degrees
- moved U2 1.08 mm to (75.3, 166.8)
Connections:
- net /RX renamed Net-(T07-Pad1)
- J1 pad 4: GND -> unconnected-(J1-Pad4)
- J1 pad 6: GND -> (no net)

Commit message: rev a fab out
Parts:
- removed T00, T01, T02, T03, T04, T05, T06, T07, T49: TestPoints, receiver:TestPoint
- added C10: CAP_0603, receiver:0603, B.Cu at (59.8, 128.3)
- added C11: CAP_0603, receiver:0603, B.Cu at (42.1, 146.4)
- added C12: CAP_0603, receiver:0603, B.Cu at (53.6, 165.0)
- added C13: CAP_0603, receiver:0603, B.Cu at (37.5, 146.4)
- added C8: CAP_0603, receiver:0603, B.Cu at (38.2, 157.2)
- added C9: CAP_0603, receiver:0603, B.Cu at (59.8, 135.8)
- added R11: RES_0603, receiver:0603, B.Cu at (50.2, 163.7)
- added R12: RES_0603, receiver:0603, B.Cu at (60.5, 149.2)
- added R13: RES_0603, receiver:0603, B.Cu at (51.7, 162.1)
- added R14: RES_0603, receiver:0603, B.Cu at (51.7, 160.4)
- added R15: RES_0603, receiver:0603, B.Cu at (51.7, 155.4)
- added R16: RES_0603, receiver:0603, B.Cu at (51.7, 158.8)
- added R17: RES_0603, receiver:0603, B.Cu at (51.7, 157.1)
- added R18: RES_0603, receiver:0603, B.Cu at (51.7, 153.8)
- added R19: RES_0603, receiver:0603, B.Cu at (51.7, 152.1)
- added R20: RES_0603, receiver:0603, B.Cu at (62.2, 149.2)
- added R21: RES_0603, receiver:0603, F.Cu at (67.2, 149.5)
- added R22: RES_0603, receiver:0603, B.Cu at (51.7, 150.5)
- added R23: RES_0603, receiver:0603, B.Cu at (63.9, 149.2)
- added R8: RES_0603, receiver:0603, B.Cu at (46.8, 150.5)
- added R9: RES_0603, receiver:0603, B.Cu at (39.8, 168.1)
- added T1: TestPoints, receiver:TestPoint, F.Cu at (37.0, 168.8)
- added T18: TestPoints, receiver:TestPoint, B.Cu at (48.4, 169.4)
- added T19: TestPoints, receiver:TestPoint, B.Cu at (34.7, 172.1)
- added T2: TestPoints, receiver:TestPoint, B.Cu at (66.9, 153.5)
- added T20: TestPoints, receiver:TestPoint, B.Cu at (31.2, 172.1)
- added T22: TestPoints, receiver:TestPoint, B.Cu at (72.0, 164.1)
- added T23: TestPoints, receiver:TestPoint, F.Cu at (29.0, 152.4)
- added T24: TestPoints, receiver:TestPoint, B.Cu at (72.0, 166.6)
- added T25: TestPoints, receiver:TestPoint, B.Cu at (29.0, 152.4)
- added T26: TestPoints, receiver:TestPoint, F.Cu at (51.2, 166.4)
- added T27: TestPoints, receiver:TestPoint, F.Cu at (61.6, 167.5)
- added T28: TestPoints, receiver:TestPoint, B.Cu at (58.3, 149.2)
- added T29: TestPoints, receiver:TestPoint, B.Cu at (63.5, 162.6)
- added T3: TestPoints, receiver:TestPoint, B.Cu at (71.9, 159.0)
- added T30: TestPoints, receiver:TestPoint, B.Cu at (63.2, 159.9)
- added T34: TestPoints, receiver:TestPoint, F.Cu at (56.1, 170.3)
- added T35: TestPoints, receiver:TestPoint, F.Cu at (53.3, 170.3)
- added T36: TestPoints, receiver:TestPoint, F.Cu at (61.6, 170.3)
- added T37: TestPoints, receiver:TestPoint, B.Cu at (63.4, 168.7)
- added T38: TestPoints, receiver:TestPoint, B.Cu at (64.3, 166.4)
- added T39: TestPoints, receiver:TestPoint, F.Cu at (61.6, 162.1)
- added T4: TestPoints, receiver:TestPoint, F.Cu at (61.7, 156.7)
- added T5: TestPoints, receiver:TestPoint, B.Cu at (72.0, 161.5)
- added T6: TestPoints, receiver:TestPoint, B.Cu at (58.8, 170.3)
- added T7: TestPoints, receiver:TestPoint, F.Cu at (64.4, 133.9)
- added T8: TestPoints, receiver:TestPoint, B.Cu at (65.4, 131.8)
- added T9: TestPoints, receiver:TestPoint, B.Cu at (65.4, 134.4)
- added U3: C8051F850-A-GU, receiver:C8051F850-A-GU, B.Cu at (55.8, 168.2)
- added U4: DRV2605LDGST, receiver:DRV2605LDGST, B.Cu at (42.1, 148.1)
- C1, T40, T41: moved to F.Cu
- C6, C7, J1, R1, R10, R2, R3, R4, R5, R6, R7, T13, T21, T48, U2: moved to B.Cu
- U1: value C8051F850-A-GU -> MPU-6050; footprint receiver:C8051F850-A-GU -> Sensor_Motion:InvenSense_QFN-24_4x4mm_P0.5mm; moved to B.Cu
- moved T45 61.6 mm to (34.3, 129.7), turned to 180 degrees
- moved T44 57.9 mm to (34.3, 137.8), turned to 180 degrees
- moved C3 53.5 mm to (62.0, 135.5), turned to 0 degrees
- moved C5 52.9 mm to (57.1, 133.2), turned to 180 degrees
- moved T46 52.8 mm to (34.3, 143.5), turned to 180 degrees
- moved T47 50.6 mm to (34.3, 135.3), turned to 180 degrees
- moved T13 45.8 mm to (41.9, 127.1), turned to 180 degrees
- moved T48 42.3 mm to (34.3, 127.1), turned to 180 degrees
- moved R2 41.5 mm to (59.7, 143.5), turned to 180 degrees
- moved R1 39.8 mm to (63.7, 143.5), turned to 180 degrees
- moved T32 39.2 mm to (58.3, 146.7)
- moved T31 38.4 mm to (53.6, 152.1)
- moved T12 37.2 mm to (41.9, 135.4)
- moved T17 34.3 mm to (27.9, 168.3)
- moved T16 34.2 mm to (27.9, 171.7)
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Connections:
- net Net-(U2-Pad15) renamed /D+
- net Net-(U2-Pad16) renamed /D-
- C3 pad 1: +5V -> +3V3
- C4 pad 1: +3V3 -> +5V
- C5 pad 1: +5V -> +3V3
- C7 pad 1: +3V3 -> +5V
- J1 pad 4: unconnected-(J1-Pad4) -> Net-(J1-Pad4)
- R1 pad 2: Net-(R1-Pad2) -> /MPU_AD0
- R10 pad 1: /TDI_C2CK -> Vdrive
- R2 pad 1: Net-(R2-Pad1) -> /MPU_AD0
- R2 pad 2: +3V3 -> GND
- T10 pad 1: Net-(T10-Pad1) -> Vdrive
- T11 pad 1: Net-(T11-Pad1) -> Vdrive
- T12 pad 1: Net-(T12-Pad1) -> Vdrive
- T13 pad 1: Net-(T13-Pad1) -> Vdrive
- T14 pad 1: Net-(T14-Pad1) -> +5V
- T15 pad 1: Net-(T15-Pad1) -> +5V
- T16 pad 1: Net-(T16-Pad1) -> +5V
- T17 pad 1: Net-(T17-Pad1) -> +5V
- T21 pad 1: Net-(T21-Pad1) -> +3V3
- T31 pad 1: /USB_PWR -> /SDA
- T32 pad 1: /TDO_C2D -> /SCL
- T33 pad 1: /TMS_C2CK -> Net-(T33-Pad1)
- T40 pad 1: +5V -> Net-(T40-Pad1)
- T41 pad 1: +5V -> Net-(T41-Pad1)
- T42 pad 1: +3V3 -> Net-(T42-Pad1)
- T43 pad 1: +3V3 -> /OUT-
- T44 pad 1: /TDI_C2CK -> /OUT-
- T45 pad 1: /TDI_C2CK -> /OUT-
- T46 pad 1: /TCK_C2D -> /OUT+
- T47 pad 1: /TCK_C2D -> /OUT+
- T48 pad 1: GND -> /OUT+
- U1 pad 1: unconnected-(U1-Pad1) -> GND
- U1 pad 10: Net-(T16-Pad1) -> Net-(C9-Pad1)
- U1 pad 11: Net-(T15-Pad1) -> GND
- U1 pad 12: Net-(T21-Pad1) -> /MPU_INT
- U1 pad 13: unconnected-(U1-Pad13) -> +3V3
- U1 pad 14: Net-(T14-Pad1) -> unconnected-(U1-Pad14)
- U1 pad 15: Net-(T13-Pad1) -> unconnected-(U1-Pad15)
- U1 pad 16: Net-(T12-Pad1) -> unconnected-(U1-Pad16)
- U1 pad 17: Net-(T11-Pad1) -> unconnected-(U1-Pad17)
- U1 pad 18: Net-(T10-Pad1) -> GND
- U1 pad 19: Net-(T07-Pad1) -> unconnected-(U1-Pad19)
- U1 pad 2: Net-(T02-Pad1) -> unconnected-(U1-Pad2)
- U1 pad 21: /FT_TO_MCU -> unconnected-(U1-Pad21)
- U1 pad 22: /MCU_TO_FT -> unconnected-(U1-Pad22)
- U1 pad 23: Net-(T03-Pad1) -> /MPU_SCL
- U1 pad 24: unconnected-(U1-Pad24) -> /MPU_SDA
- U1 pad 3: Net-(T01-Pad1) -> unconnected-(U1-Pad3)
- U1 pad 4: Net-(T00-Pad1) -> unconnected-(U1-Pad4)
- U1 pad 5: GND -> unconnected-(U1-Pad5)
- U1 pad 6: +3V3 -> Net-(T8-Pad1)
- U1 pad 7: /TDI_C2CK -> Net-(T9-Pad1)
- U1 pad 8: /TCK_C2D -> +3V3
- U1 pad 9: Net-(T17-Pad1) -> /MPU_AD0
- U2 pad 10: Net-(R6-Pad1) -> Net-(R9-Pad1)
- U2 pad 11: Net-(R3-Pad1) -> Net-(R4-Pad1)
- U2 pad 14: Net-(R1-Pad2) -> Net-(R5-Pad1)
- U2 pad 2: Net-(R4-Pad1) -> Net-(R6-Pad1)
- U2 pad 3: Net-(R2-Pad1) -> Net-(R3-Pad1)
- U2 pad 6: Net-(R7-Pad1) -> Net-(R11-Pad1)
- U2 pad 9: Net-(R5-Pad1) -> Net-(R7-Pad1)
Routing:
- net GND: track 0.00 -> 217.9 mm, vias 0 -> 97
- net +3V3: track 0.00 -> 134.8 mm, vias 0 -> 24
- net +5V: track 0.00 -> 57.6 mm, vias 0 -> 8
- net Vdrive: track 0.00 -> 55.2 mm
- net /SDA: track 0.00 -> 48.2 mm, vias 0 -> 4
- net /SCL: track 0.00 -> 45.9 mm, vias 0 -> 2
- net /TDI_C2CK: track 0.00 -> 40.7 mm, vias 0 -> 3
- net /OUT+: track 0.00 -> 32.2 mm
- net /MPU_SCL: track 0.00 -> 31.8 mm, vias 0 -> 2
- net /MPU_SDA: track 0.00 -> 29.2 mm, vias 0 -> 2
- net /MPU_INT: track 0.00 -> 27.2 mm, vias 0 -> 2
- net /OUT-: track 0.00 -> 25.7 mm
- net /FT_TO_MCU: track 0.00 -> 24.3 mm, vias 0 -> 2
- net /INT: track 0.00 -> 23.9 mm, vias 0 -> 2
- net /MCU_TO_FT: track 0.00 -> 23.1 mm, vias 0 -> 2
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- added copper zone on F.Cu, net (none)
- added copper zone on B.Cu, net +3V3
- added copper zone on F.Cu, net +3V3
- added copper zone on B.Cu, net +5V
- added copper zone on F.Cu, net +5V
- added copper zone on B.Cu, net /OUT+
- added copper zone on B.Cu, net /OUT-
- added copper zone on B.Cu, net GND
- added copper zone on F.Cu, net GND
- added copper zone on B.Cu, net Net-(C11-Pad1)
- added copper zone on B.Cu, net Vdrive
Other:
- board outline added: 49.5 x 49.5 mm
- board text added: "Dec 2023 Rev A"
- board text removed: "Dec 2021 Rev A"
