File: hardware/rev_b/BalanceBoard/BalanceBoard.kicad_sch (KiCad schematic)
At the start: 26 parts, among them T1 TestPoints, T7 TestPoints, T8 TestPoints, T9 TestPoints, U1 MPU-6050, U2 FT232RL

Commit message: add batt + LDO
Parts:
- added C11, C12, C13: CAP_0603, receiver:0603, symbol BalanceBoard-rescue:CAP_0603-receiver
- added U4: MCP73831/2, BalanceBoard:MCP738312, symbol BalanceBoard:MCP73831/2
- added U5: MIC5239-3.3YS, receiver:MIC5239-3.3YS, symbol BalanceBoard:MIC5239-3.3YS
- C8: Capacitance 100nF -> 4.7uF
- U3: renamed from U?; footprint (none) -> BalanceBoard:ESP32-WROOM-32D
Connections:
- net +3V3: now also C13.1, U5.3 (OUT); no longer C8.1, U2.17 (3V3OUT)
- net +5V: now also C11.1, U4.4 (VDD)
- net GND: now also C11.2, C12.2, C13.2, U4.2 (VSS), U5.2 (GND), U5.4 (GND)
- new net +BATT: C12.1, C8.1, U4.3 (VBAT), U5.1 (IN)
- no-connect marks 9 -> 10
Other:
- note added: "Power Supply"
- moved on the sheet: C3, C5, R1, R2

Commit message: Update schematic
Parts:
- added C14, C15, C16, C17, C18, C19, C20, C21, C22, C23, C24: CAP_0603, receiver:0603, symbol BalanceBoard-rescue:CAP_0603-receiver
- added J1: 48037-0001, receiver:48037-0001, symbol BalanceBoard:48037-0001
- added R10, R12, R13, R14, R8: RES_0603, receiver:0603, symbol BalanceBoard-rescue:RES_0603-receiver
- added T10, T11, T12, T13, T14, T15, T16, T17, T18, T2, T3, T4, T5, T6: TestPoints, receiver:TestPoint, symbol BalanceBoard-rescue:TestPoints-receiver
- added U6: TB6612FNG, receiver:TB6612FNG, symbol BalanceBoard:TB6612FNG
- added U7: MIC5239-3.3YS, receiver:MIC5239-3.3YS, symbol BalanceBoard:MIC5239-3.3YS
Connections:
- net FT_TO_MCU is gone; now on net FT_TO_ESP: U2.1 (TXD)
- net MCU_TO_FT is gone; now on net ESP_TO_FT: U2.5 (RXD)
- net +3V3: now also R11.1, R9.1, U3.2 (3V3), C15.1, C16.1, C19.1, C20.1, C21.1, R10.2, R8.2, U6.20 (VCC); no longer R11.2, R9.2
- net +5V: now also J1.1 (VCC)
- net +BATT: now also C17.1, U7.1 (IN)
- net D+: now also J1.3 (USBDP)
- net D-: now also J1.2 (USBDM)
- net GND: now also U3.1 (GND1), U3.15 (GND2), U3.38 (GND3), U3.39 (P_GND), C14.2, C15.2, C16.2, C17.2, C18.2, C19.2, C20.2, C21.2, J1.4 (GND), J1.5 (GND), J1.6 (GND), R12.1, R13.2, R14.2, U6.18 (GND), U7.2 (GND), U7.4 (GND)
- net MPU_SCL: now also U3.10 (IO25)
- net MPU_SDA: now also U3.11 (IO26)
- net at U2.10 (DCD#): now also R9.2; no longer R9.1
- net at U2.6 (RI#): now also R11.2; no longer R11.1
- net STAT: now reaches U4.1 (STAT)
- net STAT: now also R10.1
- net PROG: now reaches U4.5 (PROG)
- net PROG: now also R12.2
- net PWMB: now reaches U3.26 (IO4)
- net PWMB: now also T16.1, U6.15 (PWMB)
- net BIN2: now reaches U3.27 (IO16)
- net BIN2: now also T15.1, U6.16 (BIN2)
- net BIN1: now reaches U3.28 (IO17)
- net BIN1: now also T14.1, U6.17 (BIN1)
- net PWMA: now reaches U3.29 (IO5)
- net PWMA: now also T3.1, U6.23 (PWMA)
- net EN: now reaches U3.3 (EN)
- net EN: now also C14.1, R8.1
- net AIN2: now reaches U3.30 (IO18)
- net AIN2: now also T2.1, U6.22 (AIN2)
- net AIN1: now reaches U3.31 (IO19)
- net AIN1: now also T1.1, U6.21 (AIN1)
- net STBY: now reaches U3.33 (IO21)
- net STBY: now also T13.1, U6.19 (STBY)
- net FT_TO_ESP: now reaches U3.34 (RXD0)
- net ESP_TO_FT: now reaches U3.35 (TXDO)
- new net: T10.1, T12.1, T5.1, U6.5 (AO2), U6.6 (AO2)
- new net: T11.1, T4.1, T6.1, U6.1 (AO1), U6.2 (AO1)
- new net: T17.1, U6.11 (BO1), U6.12 (BO1)
- new net: T18.1, U6.7 (BO2), U6.8 (BO2)
- new net GND2: C22.2, C23.2, C24.2, R13.1, R14.1, U6.10 (PGND2), U6.3 (PGND1), U6.4 (PGND1), U6.9 (PGND2)
- new net Vdrive: C18.1, C22.1, C23.1, C24.1, U6.13 (VM2), U6.14 (VM3), U6.24 (VM1), U7.3 (OUT)
- no-connect marks 10 -> 31
Other:
- note added: "2K -> 500mA"
- note added: "LDOs"
- note added: "MCU + WiFi Module"
- note added: "USB Charger"
- note removed: "Power Supply"
- note removed: "USB Conn"
- moved on the sheet: C1, C10, C11, C12, C13, C2, C3, C4, C5, C6, C7, C8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

Commit message: Rev B fab out
Parts:
- removed C1, C2, C4, C6, C7: CAP_0603, receiver:0603, symbol BalanceBoard-rescue:CAP_0603-receiver
- removed J1: 48037-0001, receiver:48037-0001, symbol BalanceBoard:48037-0001
- removed R11, R9: RES_0603, receiver:0603, symbol BalanceBoard-rescue:RES_0603-receiver
- removed U2: FT232RL, receiver:FT232RL, symbol BalanceBoard-rescue:FT232RL-receiver
- added C8: CAP_0603, receiver:0603, symbol BalanceBoard-rescue:CAP_0603-receiver
- added J1: 61300611121, BalanceBoard:61300611121, symbol BalanceBoard:61300611121
- added M1, M2, M3, M4, M5, M6: MountingHole, receiver:MountingHole, symbol BalanceBoard:MountingHole
- added R8: RES_0603, receiver:0603, symbol BalanceBoard-rescue:RES_0603-receiver
- added T11, T20, T21: TestPoints, receiver:TestPoint, symbol BalanceBoard-rescue:TestPoints-receiver
- added U4: S2B-PH-SM4-TB, BalanceBoard:S2B-PH-SM4-TB, symbol BalanceBoard:S2B-PH-SM4-TB
- added U5: LP653042, BalanceBoard:LP653042, symbol BalanceBoard:LP653042
- R3, R4, R7: Resistance 10K -> DNF
- R5, R6: Resistance 10K -> 0R
- renumbered C8 to C1, C11 to C10, C19 to C11, C20 to C13, C15 to C14, C21 to C15, C14 to C16, C16 to C17, C22 to C18, C23 to C19, C17 to C2, C24 to C20, C13 to C4, C18 to C5, C9 to C6, C10 to C7, C5 to C9, R12 to R10, R13 to R11, R14 to R12, R8 to R13, R10 to R9, T7 to T1, T16 to T10, T17 to T12, T18 to T13, T4 to T14, T5 to T15, T6 to T16, T10 to T17, T11 to T18, T12 to T19, T8 to T2, T9 to T3, T13 to T4, T1 to T5, T2 to T6, T3 to T7, T14 to T8, T15 to T9, U5 to U1, U7 to U2, U1 to U3, U4 to U6, U6 to U7, U3 to U8
Connections:
- net ESP_TO_FT is gone; now on net TXD0: U8.35 (TXDO)
- net FT_TO_ESP is gone; now on net RXD0: U8.34 (RXD0)
- net +3V3: now also R4.1; no longer R4.2, R5.2, R6.2, R7.2
- net +5V: now also J1.3 (VCC)
- net +BATT: now also R7.1, U4.2 (+)
- net GND: now also C8.2, J1.1 (GND), R8.2, U4.1 (-)
- net MPU_SCL: now also R4.2
- net MPU_SDA: now also R3.1
- net STAT: now also U8.14 (IO12)
- net TXD0: now reaches R5.1
- net RXD0: now reaches R6.1
- net AO2: now reaches T15.1, T17.1, T19.1, U7.5 (AO2), U7.6 (AO2)
- net AO1: now reaches T14.1, T16.1, T18.1, U7.1 (AO1), U7.2 (AO1)
- net BO1: now reaches T12.1, U7.11 (BO1), U7.12 (BO1)
- net BO2: now reaches T13.1, U7.7 (BO2), U7.8 (BO2)
- net at U8.12 (IO27): now also T11.1
- net at U8.23 (IO15): now also T20.1
- net at U8.36 (IO22): now also T21.1
- net MEASURE: now reaches U8.7 (IO35)
- net MEASURE: now also R7.2, C8.1, R8.1
- new net: J1.4 (TXD), R6.2
- new net: J1.5 (RXD), R5.2
- new net MT: M1.1, M2.1, M3.1, M4.1, M5.1, M6.1
- no-connect marks 31 -> 20
Other:
- note added: "Battery"
- note added: "Charger"
- note added: "UART"
- note removed: "USB Charger"
- note removed: "USB to UART"
- moved on the sheet: C10, C12, C2, C5, C7, R10, R9, U2, U6
